File: pcb/_restore_backup_2026-07-21T23-03-08-659/kicad-pcb.kicad_sch (KiCad schematic)
At the start: 25 parts, among them J1 InputJack, J2 OutputJack, J3 Power Jack, U2 LM7805_TO220

Commit message: pcb complete
Parts:
- removed D3: LED, LED_THT:LED_D3.0mm, symbol Device:LED
- removed R7: 150, Resistor_THT:R_Axial_DIN0207_L6.3mm_D2.5mm_P7.62mm_Horizontal, symbol Device:R_Small
- removed SW1: (no value), GuitarPedal:Switches_Stomp_Switch_3PDT, symbol GuitarPedal:3PDT_Switch
- removed U6: (no value), GuitarPedal:Mini_F4X1_STM32, symbol GuitarPedal:STM32_BlackPill
- added SW1: OnOff, symbol Switch:SW_SPST
- added U4: (no value), symbol GuitarPedal:STM32F411_Black_Pill
- C1: footprint Capacitor_THT:C_Disc_D10.0mm_W2.5mm_P5.00mm -> (none)
- C2: footprint Capacitor_THT:CP_Radial_D6.3mm_P2.50mm -> (none)
- C3, C4: footprint Capacitor_THT:CP_Radial_D5.0mm_P2.00mm -> (none)
- J1, J2: footprint GuitarPedal:AudioJack -> (none)
- J2: renamed from J3; footprint Connector_BarrelJack:BarrelJack_Horizontal -> (none)
- R1, R2, R3, R4, R5: footprint Resistor_THT:R_Axial_DIN0207_L6.3mm_D2.5mm_P7.62mm_Horizontal -> (none)
- RV1, RV2, RV3: footprint Potentiometer_THT:Potentiometer_Alps_RK09K_Single_Vertical -> (none)
- U1: footprint GuitarPedal:DIP787W46P254L927H533Q8 -> (none)
- U3: footprint GuitarPedal:pcm_adc -> (none)
- U5: footprint GuitarPedal:GY-PCM5102 -> (none)
Connections:
- net +3.3V: now also SW1.2 (B), U4.1 (3v3), U4.2 (3v3); no longer RV1.1, RV2.1, RV3.1
- net +5V: now also U4.3 (5V), U4.4 (5V)
- net GND: now also U4.5 (GND), U4.6 (GND)
- net at J2.T: now also U5.15 (L)
- net at U3.12 (LRC), U5.4 (LCK): now also U4.6 (GND)
- net at U3.10 (BCK), U5.2 (BCK): now also U4.17 (B3)
- net at U3.11 (OUT): now also U4.18 (B4)
- net at U5.3 (DIN): now also U4.19 (B5)
- net at U3.13 (SCK): now also U4.24 (B10)
- net at R5.2: now also R4.1, U1.2 (-); no longer C3.1
- net at C4.1, U1.3: now also R4.2; no longer R4.1
- net at U3.3 (LIN): now also C4.2, D1.2 (A), D2.1 (K)
- new net: SW1.1 (A), U4.28 (A7)
- new net: C3.1, R5.1
Other:
- moved on the sheet: D1, D2, J2, RV1, U3
